File: hardware/electrical/artsey_ergo.kicad_pcb (KiCad board)
At the start: 2 copper layers, 94 x 57.8 mm, 41 parts

Commit message: Fix clearance issues with battery connector and ground fill
Routing:
- net GND: track 64.8 -> 59.9 mm
