File: hardware/electrical/artsey_ergo.kicad_pcb (KiCad board)
At the start: 2 copper layers, 94 x 57.8 mm, 41 parts

Commit message: Move LED data and I2C pins to high speed pin to avoid RF interference
Parts:
- moved REF** 0.70 mm to (247.9, 135.0) (x2)
- moved kibuzzard-67450C30 0.10 mm to (170.4, 175.1)
- moved kibuzzard-67450C3F 0.10 mm to (169.0, 175.1)
Connections:
- MCU1 pad 101: P1 -> LED_DIN
- MCU1 pad 19: key_matrix_index_top -> MCU1_19
- MCU1 pad 20: key_matrix_middle_top -> MCU1_20
- MCU1 pad 5: OLED_SDA -> MCU1_5
- MCU1 pad 6: OLED_SCL -> MCU1_6
- MCU1 pad 8: LED_DIN -> P5
Routing:
- net LED_DIN: track 29.5 -> 52.2 mm
- net key_matrix_index_top: track 6.46 -> 21.2 mm
- net key_matrix_middle_top: track 25.0 -> 39.2 mm
- net P1: track 10.2 -> 0.00 mm
- net OLED_SCL: track 28.7 -> 38.6 mm
- net OLED_SDA: track 35.3 -> 44.7 mm, vias 1 -> 2
- net MCU1_20: track 0.00 -> 4.25 mm
- net MCU1_19: track 0.00 -> 4.25 mm
- net MCU1_6: track 0.00 -> 4.23 mm
- net MCU1_5: track 0.00 -> 4.23 mm
- net RAW: track 54.2 -> 56.9 mm
- net GND: vias 121 -> 117

Commit message: Clean up and modify PCB, create Schematic, prepare for documentation generation
Parts:
- removed H1, H2, H3, H4: , ceoloide:mounting_hole_plated
- removed kibuzzard-67450C30 (x2): G***, kibuzzard-67450C30
- removed kibuzzard-67450C3F (x2): G***, kibuzzard-67450C3F
- removed kibuzzard-67450C96 (x2): G***, kibuzzard-67450C96
- removed kibuzzard-67450D2D (x2): G***, kibuzzard-67450D2D
- removed kibuzzard-67450D58 (x2): G***, kibuzzard-67450D58
- removed kibuzzard-67450FBF (x2): G***, kibuzzard-67450FBF
- added REF**: Artsey_Logo, Artsey_Ergo:Artsey_Logo, F.Cu at (112.5, 131.4)
- added REF**: blahaj, Artsey_Ergo:blahaj, F.Cu at (103.8, 110.8)
- added REF**: version, Artsey_Ergo:version, F.Cu at (130.5, 120.5)
- added REF**: engineer, Artsey_Ergo:engineer, F.Cu at (148.5, 113.2)
- CN1: renamed from JST1; value (none) -> JST PH 2.0mm 1x2; footprint ceoloide:battery_connector_jst_ph_2 -> Artsey_Ergo:battery_connector_jst_ph_2
- DP1: renamed from DISP1; value (none) -> 128x32 monochrome OLED; footprint ceoloide:display_ssd1306 -> Artsey_Ergo:display_ssd1306
- K1: renamed from S2; value (none) -> Kailh Choc Hotswap; footprint ceoloide:switch_choc_v1_v2 -> Artsey_Ergo:switch_choc_v1_v2
- K2: renamed from S4; value (none) -> Kailh Choc Hotswap; footprint ceoloide:switch_choc_v1_v2 -> Artsey_Ergo:switch_choc_v1_v2
- K3: renamed from S6; value (none) -> Kailh Choc Hotswap; footprint ceoloide:switch_choc_v1_v2 -> Artsey_Ergo:switch_choc_v1_v2
- K4: renamed from S8; value (none) -> Kailh Choc Hotswap; footprint ceoloide:switch_choc_v1_v2 -> Artsey_Ergo:switch_choc_v1_v2
- K5: renamed from S1; value (none) -> Kailh Choc Hotswap; footprint ceoloide:switch_choc_v1_v2 -> Artsey_Ergo:switch_choc_v1_v2
- K6: renamed from S3; value (none) -> Kailh Choc Hotswap; footprint ceoloide:switch_choc_v1_v2 -> Artsey_Ergo:switch_choc_v1_v2
- K7: renamed from S5; value (none) -> Kailh Choc Hotswap; footprint ceoloide:switch_choc_v1_v2 -> Artsey_Ergo:switch_choc_v1_v2
- K8: renamed from S7; value (none) -> Kailh Choc Hotswap; footprint ceoloide:switch_choc_v1_v2 -> Artsey_Ergo:switch_choc_v1_v2
- L1: renamed from LED5; value (none) -> SK6812MINI-E; footprint ceoloide:led_SK6812mini-e (per-key, reversible) -> Artsey_Ergo:led_SK6812mini-e (per-key, reversible)
- L2: renamed from LED6; value (none) -> SK6812MINI-E; footprint ceoloide:led_SK6812mini-e (per-key, reversible) -> Artsey_Ergo:led_SK6812mini-e (per-key, reversible)
- L3: renamed from LED7; value (none) -> SK6812MINI-E; footprint ceoloide:led_SK6812mini-e (per-key, reversible) -> Artsey_Ergo:led_SK6812mini-e (per-key, reversible)
- L4: renamed from LED8; value (none) -> SK6812MINI-E; footprint ceoloide:led_SK6812mini-e (per-key, reversible) -> Artsey_Ergo:led_SK6812mini-e (per-key, reversible)
- L5: renamed from LED1; value (none) -> SK6812MINI-E; footprint ceoloide:led_SK6812mini-e (per-key, reversible) -> Artsey_Ergo:led_SK6812mini-e (per-key, reversible)
- L6: renamed from LED2; value (none) -> SK6812MINI-E; footprint ceoloide:led_SK6812mini-e (per-key, reversible) -> Artsey_Ergo:led_SK6812mini-e (per-key, reversible)
- L7: renamed from LED3; value (none) -> SK6812MINI-E; footprint ceoloide:led_SK6812mini-e (per-key, reversible) -> Artsey_Ergo:led_SK6812mini-e (per-key, reversible)
- L8: renamed from LED4; value (none) -> SK6812MINI-E; footprint ceoloide:led_SK6812mini-e (per-key, reversible) -> Artsey_Ergo:led_SK6812mini-e (per-key, reversible)
- MCU1: value (none) -> Pro Micro Compatible MCU; footprint ceoloide:mcu_nice_nano -> Artsey_Ergo:mcu_nice_nano
- MH1, MH2: value (none) -> Mounting Hole; footprint ceoloide:mounting_hole_npth -> Artsey_Ergo:mounting_hole
- RS1: renamed from RST1; value (none) -> EVQ-PUA02K; footprint ceoloide:reset_switch_smd_side -> Artsey_Ergo:reset_switch_smd_side
- SW1: renamed from PWR1; value (none) -> Alps SSSS811101; footprint ceoloide:power_switch_smd_side -> Artsey_Ergo:power_switch_smd_side
- moved CN1 75.3 mm to (144.5, 117.6)
- moved DP1 75.3 mm to (187.6, 99.8)
- moved K1 75.3 mm to (112.5, 105.0)
- moved K2 75.3 mm to (130.5, 93.0)
- moved K3 75.3 mm to (148.5, 87.0)
- moved K4 75.3 mm to (166.5, 93.0)
- moved K5 75.3 mm to (112.5, 123.0)
- moved K6 75.3 mm to (130.5, 111.0)
- moved K7 75.3 mm to (148.5, 105.0)
- moved K8 75.3 mm to (166.5, 111.0)
- moved MH1 75.3 mm to (121.0, 114.0)
- moved MH2 75.3 mm to (157.0, 96.0)
- moved REF** 75.3 mm to (186.4, 91.5) (x2)
- moved RS1 75.3 mm to (166.5, 79.0)
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Connections:
- CN1 pad 1: BAT_P -> Net-(CN1-Pin_1)
- CN1 pad 11: JST1_1 -> unconnected-(CN1-Pad11)
- CN1 pad 12: JST1_2 -> unconnected-(CN1-Pad12)
- DP1 pad 1: DISP1_1 -> /Block Diagram/Display/SDA
- DP1 pad 2: DISP1_2 -> /Block Diagram/Display/SCL
- DP1 pad 21: DISP1_3 -> unconnected-(DP1-Pad21)
- DP1 pad 22: DISP1_2 -> unconnected-(DP1-Pad22)
- DP1 pad 23: DISP1_1 -> unconnected-(DP1-Pad23)
- DP1 pad 24: GND -> unconnected-(DP1-Pad24)
- DP1 pad 3: DISP1_3 -> /Block Diagram/Display/VCC
- DP1 pad 4: DISP1_4 -> GND
- K1 pad 1: GND -> /Block Diagram/MCU/K1
- K1 pad 2: key_matrix_pinky_top -> GND
- K2 pad 1: GND -> /Block Diagram/MCU/K2
- K2 pad 2: key_matrix_ring_top -> GND
- K3 pad 1: GND -> /Block Diagram/MCU/K3
- K3 pad 2: key_matrix_middle_top -> GND
- K4 pad 1: GND -> /Block Diagram/MCU/K4
- K4 pad 2: key_matrix_index_top -> GND
- K5 pad 1: GND -> /Block Diagram/MCU/K5
- K5 pad 2: key_matrix_pinky_home -> GND
- K6 pad 1: GND -> /Block Diagram/MCU/K6
- K6 pad 2: key_matrix_ring_home -> GND
- K7 pad 1: GND -> /Block Diagram/MCU/K7
- K7 pad 2: key_matrix_middle_home -> GND
- K8 pad 1: GND -> /Block Diagram/MCU/K8
- K8 pad 2: key_matrix_index_home -> GND
- L1 pad 1: VCC -> Net-(L1-DOUT)
- L1 pad 2: led_matrix_pinky_home -> GND
- L1 pad 3: GND -> Net-(L1-DIN)
- L1 pad 4: led_matrix_pinky_top -> /Block Diagram/Display/VCC
- L2 pad 1: VCC -> Net-(L1-DIN)
- L2 pad 2: led_matrix_pinky_top -> GND
- L2 pad 3: GND -> Net-(L2-DIN)
- L2 pad 4: led_matrix_ring_top -> /Block Diagram/Display/VCC
- L3 pad 1: VCC -> Net-(L2-DIN)
- L3 pad 2: led_matrix_ring_top -> GND
- L3 pad 3: GND -> Net-(L3-DIN)
- L3 pad 4: led_matrix_middle_top -> /Block Diagram/Display/VCC
- L4 pad 1: VCC -> Net-(L3-DIN)
- L4 pad 2: led_matrix_middle_top -> GND
- L4 pad 3: GND -> /Block Diagram/LEDs/DIN
- L4 pad 4: LED_DIN -> /Block Diagram/Display/VCC
- L5 pad 1: VCC -> Net-(L5-DOUT)
- L5 pad 2: led_matrix_ring_home -> GND
- L5 pad 3: GND -> Net-(L1-DOUT)
- L5 pad 4: led_matrix_pinky_home -> /Block Diagram/Display/VCC
- L6 pad 1: VCC -> Net-(L6-DOUT)
- L6 pad 2: led_matrix_middle_home -> GND
- L6 pad 3: GND -> Net-(L5-DOUT)
- L6 pad 4: led_matrix_ring_home -> /Block Diagram/Display/VCC
- L7 pad 1: VCC -> Net-(L7-DOUT)
- L7 pad 2: led_matrix_index_home -> GND
- L7 pad 3: GND -> Net-(L6-DOUT)
- L7 pad 4: led_matrix_middle_home -> /Block Diagram/Display/VCC
- L8 pad 1: VCC -> unconnected-(L8-DOUT-Pad1)
- L8 pad 2: x -> GND
- L8 pad 3: GND -> Net-(L7-DOUT)
- L8 pad 4: led_matrix_index_home -> /Block Diagram/Display/VCC
- MCU1 pad 1: MCU1_1 -> unconnected-(MCU1-TX0/PD3-Pad1)
- MCU1 pad 10: P7 -> unconnected-(MCU1-7/PE6-Pad10)
- MCU1 pad 101: LED_DIN -> unconnected-(MCU1-Pad101)
- MCU1 pad 102: P0 -> unconnected-(MCU1-Pad102)
- MCU1 pad 103: GND -> unconnected-(MCU1-Pad103)
- MCU1 pad 104: GND -> unconnected-(MCU1-Pad104)
- MCU1 pad 105: OLED_SDA -> unconnected-(MCU1-Pad105)
- MCU1 pad 106: OLED_SCL -> unconnected-(MCU1-Pad106)
- MCU1 pad 11: P8 -> unconnected-(MCU1-8/PB4-Pad11)
- MCU1 pad 119: key_matrix_index_top -> unconnected-(MCU1-Pad119)
- MCU1 pad 12: P9 -> unconnected-(MCU1-9/PB5-Pad12)
- MCU1 pad 120: key_matrix_middle_top -> unconnected-(MCU1-Pad120)
- MCU1 pad 121: VCC -> unconnected-(MCU1-Pad121)
- MCU1 pad 122: RST -> unconnected-(MCU1-Pad122)
- MCU1 pad 123: GND -> unconnected-(MCU1-Pad123)
- MCU1 pad 124: RAW -> unconnected-(MCU1-Pad124)
- MCU1 pad 13: key_matrix_index_home -> /Block Diagram/MCU/K8
- MCU1 pad 14: key_matrix_pinky_home -> /Block Diagram/MCU/K5
- MCU1 pad 15: key_matrix_ring_home -> /Block Diagram/MCU/K6
- MCU1 pad 16: key_matrix_middle_home -> /Block Diagram/MCU/K7
- MCU1 pad 17: key_matrix_pinky_top -> /Block Diagram/MCU/K1
- MCU1 pad 18: key_matrix_ring_top -> /Block Diagram/MCU/K2
- MCU1 pad 19: MCU1_19 -> /Block Diagram/MCU/K4
- MCU1 pad 2: MCU1_2 -> unconnected-(MCU1-RX1/PD2-Pad2)
- MCU1 pad 20: MCU1_20 -> /Block Diagram/MCU/K3
- MCU1 pad 21: MCU1_21 -> /Block Diagram/Display/VCC
- MCU1 pad 22: MCU1_22 -> /Block Diagram/MCU/RESET
- MCU1 pad 23: MCU1_23 -> GND
- MCU1 pad 24: MCU1_24 -> /Block Diagram/Battery/RAW
- MCU1 pad 3: MCU1_3 -> GND
- MCU1 pad 4: MCU1_4 -> GND
- MCU1 pad 5: MCU1_5 -> /Block Diagram/Display/SDA
- MCU1 pad 6: MCU1_6 -> /Block Diagram/Display/SCL
- MCU1 pad 7: P4 -> unconnected-(MCU1-4/PD4-Pad7)
- MCU1 pad 8: P5 -> /Block Diagram/LEDs/DIN
- MCU1 pad 9: P6 -> unconnected-(MCU1-6/PD7-Pad9)
- RS1 pad 1: GND -> /Block Diagram/MCU/RESET
- RS1 pad 2: RST -> GND
- SW1 pad 1: BAT_P -> /Block Diagram/Battery/RAW
- SW1 pad 2: RAW -> Net-(CN1-Pin_1)
- SW1 pad 3: BAT_P -> unconnected-(SW1-C-Pad3)
Routing:
- net VCC: track 340.4 -> 0.00 mm, vias 12 -> 0
- net /Block Diagram/Display/VCC: track 0.00 -> 339.7 mm, vias 0 -> 12
- net /Block Diagram/MCU/K5: track 0.00 -> 66.7 mm
- net key_matrix_pinky_home: track 66.7 -> 0.00 mm
- net /Block Diagram/MCU/K1: track 0.00 -> 66.6 mm
- net key_matrix_pinky_top: track 66.6 -> 0.00 mm
- net /Block Diagram/Battery/RAW: track 0.00 -> 56.9 mm, vias 0 -> 1
- net RAW: track 56.9 -> 0.00 mm, vias 1 -> 0
- net LED_DIN: track 52.2 -> 0.00 mm, vias 3 -> 0
- net key_matrix_ring_top: track 48.3 -> 0.00 mm
- net /Block Diagram/MCU/K2: track 0.00 -> 48.3 mm
- net OLED_SDA: track 44.7 -> 0.00 mm, vias 2 -> 0
- net /Block Diagram/Display/SDA: track 0.00 -> 44.0 mm, vias 0 -> 2
- net key_matrix_ring_home: track 42.9 -> 0.00 mm
- net /Block Diagram/MCU/K6: track 0.00 -> 42.9 mm
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- added copper zone on B.Cu, net /Block Diagram/Display/VCC
- added copper zone on F.Cu, net /Block Diagram/MCU/RESET
- removed copper zone on F.Cu, net RST
- removed copper zone on B.Cu, net VCC
